Commit message: Add new URDF and mesh files for the robotic arm
- Created new material file for link 6 visuals with various materials defined.
- Added OBJ file for link 6 visuals.
- Introduced new URDF file defining the robotic arm structure, including joints and links with inertial properties.
- Added a no-inertial version of the URDF for simplified simulations.
- Created a patched URDF file with corrected inertial properties for better simulation accuracy.
- Implemented Python scripts for URDF validation and inverse kinematics testing using Genesis.
- Developed a utility script to clean URDF files by removing inertial blocks and normalizing origin values.

File: assets/angle_excurate_arm_ver2_to_unity/angle_excurate_arm_ver2.urdf (robot description, URDF)
Before this commit: robot angle_excurate_arm_ver2, 9 links, 8 joints
Links:
- link base_link: geometry collision mesh filename=angle_excurate_arm_ver2_description/meshes/base_link.stl scale=0.001 0.001 0.001; visual mesh filename=angle_excurate_arm_ver2_description/meshes/base_link.stl scale=0.001 0.001 0.001
- link base_link2_v2_1: geometry collision mesh filename=angle_excurate_arm_ver2_description/meshes/base_link2_v2_1.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 scale=0.001 0.001 0.001; visual mesh filename=angle_excurate_arm_ver2_description/meshes/base_link2_v2_1.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 scale=0.001 0.001 0.001
- link base_link_2_1: geometry collision mesh filename=angle_excurate_arm_ver2_description/meshes/base_link_2_1.stl scale=0.001 0.001 0.001; visual mesh filename=angle_excurate_arm_ver2_description/meshes/base_link_2_1.stl scale=0.001 0.001 0.001
- link camera_1: geometry collision mesh filename=angle_excurate_arm_ver2_description/meshes/camera_1.stl scale=0.001 0.001 0.001; visual mesh filename=angle_excurate_arm_ver2_description/meshes/camera_1.stl scale=0.001 0.001 0.001
- link link3_v1_1: geometry collision mesh filename=angle_excurate_arm_ver2_description/meshes/link3_v1_1.stl scale=0.001 0.001 0.001; visual mesh filename=angle_excurate_arm_ver2_description/meshes/link3_v1_1.stl scale=0.001 0.001 0.001
- link link4_v1_1: geometry collision mesh filename=angle_excurate_arm_ver2_description/meshes/link4_v1_1.stl scale=0.001 0.001 0.001; visual mesh filename=angle_excurate_arm_ver2_description/meshes/link4_v1_1.stl scale=0.001 0.001 0.001
- link robot_ver7_grap1_2_v1_1: geometry collision mesh filename=angle_excurate_arm_ver2_description/meshes/robot_ver7_grap1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 scale=0.001 0.001 0.001; visual mesh filename=angle_excurate_arm_ver2_description/meshes/robot_ver7_grap1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 scale=0.001 0.001 0.001
- link robot_ver7_grap2_2_v1_1: geometry collision mesh filename=angle_excurate_arm_ver2_description/meshes/robot_ver7_grap2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 scale=0.001 0.001 0.001; visual mesh filename=angle_excurate_arm_ver2_description/meshes/robot_ver7_grap2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 scale=0.001 0.001 0.001
- link robot_ver7_link_4_v1_1: geometry collision mesh filename=angle_excurate_arm_ver2_description/meshes/robot_ver7_link_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 scale=0.001 0.001 0.001; visual mesh filename=angle_excurate_arm_ver2_description/meshes/robot_ver7_link_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 scale=0.001 0.001 0.001
